File: Hardware/PCB Design/ATMega328PCBBoard.brd (EAGLE design)
At the start: 40.3 x 19.1 mm, 14 parts

Commit message: updated board again
Parts:
- moved R2 0.32 mm to (60.6, 47.0)
Routing:
- net GND: track 60.4 -> 61.6 mm
Changed lines of the file:
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@@
 <element name="MOTOR" library="SparkFun-Connectors" package="1X04-1.5MM_JST" value="" x="74.93" y="45.72"/>
 <element name="R1" library="resistor" package="0207/2V" value="220" x="60.96" y="44.45"/>
-<element name="R2" library="resistor" package="0207/2V" value="220" x="60.96" y="46.99"/>
+<element name="R2" library="resistor" package="0207/2V" value="220" x="60.6425" y="46.99"/>
 <element name="LEDGREEN" library="SparkFun-Connectors" package="JST-2-PTH-VERT" value="" x="67.31" y="38.1" rot="R180"/>
 <element name="LEDBLUE" library="SparkFun-Connectors" package="JST-2-PTH-VERT" value="" x="60.96" y="38.1" rot="R180"/>
@@
 <wire x1="72.39" y1="49.53" x2="73.66" y2="48.26" width="0.4064" layer="1"/>
 <wire x1="73.66" y1="48.26" x2="73.66" y2="47.625" width="0.4064" layer="1"/>
-<wire x1="73.66" y1="47.625" x2="76.2" y2="47.625" width="0.4064" layer="1"/>
-<wire x1="76.2" y1="47.625" x2="76.43" y2="47.395" width="0.4064" layer="1"/>
-<wire x1="76.43" y1="47.395" x2="76.43" y2="45.72" width="0.4064" layer="1"/>
+<wire x1="73.66" y1="47.625" x2="75.8825" y2="47.625" width="0.4064" layer="1"/>
+<wire x1="75.8825" y1="47.625" x2="75.8825" y2="46.585" width="0.4064" layer="1"/>
+<wire x1="75.8825" y1="46.585" x2="76.43" y2="45.72" width="0.4064" layer="1"/>
 </signal>
 <signal name="A1">
@@
 <wire x1="61.96" y1="38.65" x2="60.96" y2="39.6025" width="0.4064" layer="1"/>
 <wire x1="60.96" y1="39.6025" x2="60.96" y2="46.99" width="0.4064" layer="1"/>
-<wire x1="60.96" y1="46.99" x2="62.23" y2="46.99" width="0.4064" layer="1"/>
+<wire x1="60.96" y1="46.99" x2="61.9125" y2="46.99" width="0.4064" layer="1"/>
 </signal>
 <signal name="GND">
@@
 <wire x1="83.82" y1="46.355" x2="83.82" y2="45.085" width="0.4064" layer="1"/>
 <via x="83.82" y="45.085" extent="1-16" drill="0.7" shape="square"/>
-<wire x1="79.43" y1="45.72" x2="79.375" y2="45.72" width="0.4064" layer="1"/>
-<wire x1="79.375" y1="45.72" x2="77.47" y2="43.815" width="0.4064" layer="1"/>
 <wire x1="79.43" y1="45.72" x2="79.43" y2="45.665" width="0.4064" layer="16"/>
 <wire x1="79.43" y1="45.665" x2="80.01" y2="45.085" width="0.4064" layer="16"/>
@@
 <wire x1="76.2" y1="41.91" x2="77.47" y2="41.91" width="0.4064" layer="1"/>
 <via x="73.3425" y="45.4025" extent="1-16" drill="0.7" shape="square"/>
-<wire x1="59.69" y1="46.99" x2="59.69" y2="45.72" width="0.4064" layer="16"/>
+<wire x1="59.3725" y1="46.99" x2="59.69" y2="45.72" width="0.4064" layer="16"/>
 <wire x1="59.69" y1="45.72" x2="62.865" y2="45.72" width="0.4064" layer="16"/>
 <wire x1="62.865" y1="45.72" x2="63.1825" y2="45.4025" width="0.4064" layer="16"/>
@@
 <wire x1="65.0875" y1="45.4025" x2="65.0875" y2="45.995" width="0.4064" layer="16"/>
 <wire x1="65.0875" y1="45.995" x2="65.945" y2="46.8525" width="0.4064" layer="16"/>
-<wire x1="59.69" y1="44.45" x2="59.69" y2="46.99" width="0.4064" layer="1"/>
+<wire x1="59.69" y1="44.45" x2="59.3725" y2="46.99" width="0.4064" layer="1"/>
 <wire x1="87.63" y1="46.355" x2="89.535" y2="44.45" width="0.4064" layer="1"/>
 <wire x1="89.535" y1="44.45" x2="88.9" y2="43.815" width="0.4064" layer="1"/>
@@
 <wire x1="93.44" y1="38.65" x2="92.44" y2="38.65" width="0.4064" layer="1"/>
 <wire x1="83.82" y1="46.355" x2="87.63" y2="46.355" width="0.4064" layer="1"/>
+<wire x1="77.47" y1="43.815" x2="79.43" y2="43.815" width="0.4064" layer="1"/>
+<wire x1="79.43" y1="43.815" x2="79.43" y2="45.72" width="0.4064" layer="1"/>
 </signal>
 <signal name="3VCC">

Commit message: final board design
Parts:
- removed LM7805: V_REG_LD1117VXX, SparkFun-PowerIC:78XXL
- added IC1: 7805TV, linear:TO220V
Connections:
- net GND: now also IC1.2; no longer LM7805.IN
- net N$4: now also IC1.1; no longer LM7805.OUT
- net VCC: now also IC1.3; no longer LM7805.GND
Routing:
- net GND: track 61.6 -> 66.0 mm, vias 2 -> 3
- net 3VCC: track 31.9 -> 35.7 mm
- net N$4: track 28.3 -> 29.0 mm
- net VCC: track 16.7 -> 17.3 mm
