File: Hardware/PCB Design/ATMega328PCBBoard.sch (EAGLE design)
At the start: 9 parts, among them U1 ATMEGA328P_PDIP

Commit message: finished pcb
Parts:
- removed BATT1: AAA, adafruit:AAA
- removed C3, C4: (no value), adafruit:C-US050-025X075
- removed U1: ATMEGA328P_PDIP, SparkFun-DigitalIC:ATMEGA328P_PDIP
- added ATMEGA: ATMEGA328P_PDIP, SparkFun-DigitalIC:ATMEGA328P_PDIP
- added BATTERY, LEDBLUE, LEDGREEN: (no value), SparkFun-Connectors:M02JST-PTH-VERT
- added JP1: (no value), SparkFun-Connectors:M05JST-VERT
- added MOTOR: (no value), SparkFun-Connectors:M04JST
- added R2: 220, resistor:R-US_0207/2V
- R1: value (none) -> 220; device resistor:R-US_0207/10 -> resistor:R-US_0207/2V
- renumbered U$1 to LM7805
Connections:
- removed net GND: BATT1.-, C1.2, C2.2, LM7805.GND, U1.GND@1
- new net 0: ATMEGA.PD0(RXD), JP1.4
- new net 1: ATMEGA.PD1(TXD), JP1.3
- new net 10: ATMEGA.PB2(SS/OC1B), MOTOR.3
- new net 11: ATMEGA.PB3(MOSI/OC2)
- new net 12: ATMEGA.PB4(MISO), LEDBLUE.2
- new net 13: ATMEGA.PB5(SCK), LEDGREEN.2
- new net 2: ATMEGA.PD2(INT0)
- new net 3: ATMEGA.PD3(INT1)
- new net 4: ATMEGA.PD4(XCK/T0)
- new net 5: ATMEGA.PD5(T1)
- new net 6: ATMEGA.PD6(AIN0)
- new net 7: ATMEGA.PD7(AIN1), JP1.1
- new net 8: ATMEGA.PB0(ICP)
- new net 9: ATMEGA.PB1(OC1A)
- new net A0: ATMEGA.PC0(ADC0), MOTOR.2
- new net A1: ATMEGA.PC1(ADC1)
- new net A2: ATMEGA.PC2(ADC2)
- new net A3: ATMEGA.PC3(ADC3)
- new net A4: ATMEGA.PC4(ADC4/SDA)
- new net A5: ATMEGA.PC5(ADC5/SCL)
- new net N$3: LEDGREEN.1, R1.2
- new net N$5: LEDBLUE.1, R2.2
- new net N$7: R2.1
- new net VCC: ATMEGA.AVCC, ATMEGA.VCC, JP1.5, LM7805.OUT, MOTOR.1
- new net XBEE2: ATMEGA.GND@1, BATTERY.1, C1.2, C2.2, JP1.2, LM7805.GND, MOTOR.4
- net N$1: now also ATMEGA.PB7(XTAL2/TOSC2); no longer U1.PB7(XTAL2/TOSC2)
- net N$2: now also ATMEGA.PB6(XTAL1/TOSC1); no longer U1.PB6(XTAL1/TOSC1)
- net N$4: now also BATTERY.2; no longer BATT1.+
- net N$6: now also R1.1; no longer LM7805.OUT, U1.AVCC, U1.VCC
Other:
- note added: "0"
- note added: "1"
- note added: "10"
- note added: "11"
- note added: "12"
- note added: "13"
- note added: "2"
- note added: "3"
- note added: "4"
- note added: "5"
- note added: "6"
- note added: "7"
- note added: "8"
- note added: "9"
- note added: "A0"
- note added: "A1"
- note added: "A2"
- note added: "A3"
- note added: "A4"
- note added: "A5"
- note added: "VCC"
- moved on the sheet: R1

Commit message: updated pcb
Parts:
- added 3.3REGULATOR: (no value), SparkFun-Connectors:M03JST-PTH-VERT
- added LOAD: (no value), SparkFun-Connectors:M02JST-PTH-VERT
- renumbered JP1 to XBEE
Connections:
- removed net N$6: R1.1
- removed net N$7: R2.1
- removed net XBEE2: ATMEGA.GND@1, BATTERY.1, C1.2, C2.2, LM7805.GND, MOTOR.4, XBEE.2
- new net 3VCC: 3.3REGULATOR.3, XBEE.5
- new net GND: 3.3REGULATOR.1, ATMEGA.GND@1, BATTERY.1, C1.2, C2.2, LM7805.GND, MOTOR.4, R1.1, R2.1, XBEE.2
- net 0: now also LOAD.1
- net 1: now also LOAD.2
- net N$4: now also 3.3REGULATOR.2
- net VCC: no longer XBEE.5

Commit message: final board design
Parts:
- removed LM7805: V_REG_LD1117VXX, SparkFun-PowerIC:V_REG_LD1117VXX
- added IC1: 7805TV, linear:7805TV
Connections:
- net GND: now also IC1.GND; no longer LM7805.GND
- net N$4: now also IC1.VI; no longer LM7805.IN
- net VCC: now also IC1.VO; no longer LM7805.OUT
Changed lines of the file:
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@@
 <part name="C1" library="adafruit" deviceset="C-US" device="050-025X075" value="22pF"/>
 <part name="C2" library="adafruit" deviceset="C-US" device="050-025X075" value="22pF"/>
-<part name="LM7805" library="SparkFun-PowerIC" deviceset="V_REG_LD1117VXX" device=""/>
 <part name="MOTOR" library="SparkFun-Connectors" deviceset="M04" device="JST"/>
 <part name="R1" library="resistor" deviceset="R-US_" device="0207/2V" value="220"/>
@@
 <part name="LOAD" library="SparkFun-Connectors" deviceset="M02" device="JST-PTH-VERT"/>
 <part name="3.3REGULATOR" library="SparkFun-Connectors" deviceset="M03" device="JST-PTH-VERT"/>
+<part name="IC1" library="linear" deviceset="78*" device="TV" technology="05"/>
 </parts>
 <sheets>
@@
 <instance part="C1" gate="G$1" x="-12.7" y="48.26"/>
 <instance part="C2" gate="G$1" x="7.62" y="48.26"/>
-<instance part="LM7805" gate="G$1" x="-15.24" y="33.02"/>
 <instance part="MOTOR" gate="G$1" x="106.68" y="66.04" rot="R180"/>
 <instance part="R1" gate="G$1" x="35.56" y="12.7"/>
@@
 <instance part="LOAD" gate="G$1" x="5.08" y="86.36"/>
 <instance part="3.3REGULATOR" gate="G$1" x="-50.165" y="47.9425"/>
+<instance part="IC1" gate="A1" x="-7.3025" y="8.5725"/>
 </instances>
 <busses>
@@
 <net name="VCC" class="0">
 <segment>
-<pinref part="LM7805" gate="G$1" pin="OUT"/>
 <wire x1="-7.62" y1="33.02" x2="12.7" y2="33.02" width="0.1524" layer="91"/>
 <wire x1="12.7" y1="33.02" x2="12.7" y2="38.1" width="0.1524" layer="91"/>
@@
 <wire x1="101.6" y1="68.58" x2="99.06" y2="68.58" width="0.1524" layer="91"/>
 </segment>
+<segment>
+<pinref part="IC1" gate="A1" pin="VO"/>
+<wire x1="2.8575" y1="8.5725" x2="6.0325" y2="8.5725" width="0.1524" layer="91"/>
+</segment>
 </net>
 <net name="A0" class="0">
@@
 <junction x="-2.54" y="40.64"/>
 <wire x1="-27.94" y1="17.78" x2="-15.24" y2="17.78" width="0.1524" layer="91"/>
-<pinref part="LM7805" gate="G$1" pin="GND"/>
 <wire x1="-15.24" y1="17.78" x2="-15.24" y2="25.4" width="0.1524" layer="91"/>
 <wire x1="-15.24" y1="17.78" x2="-2.54" y2="17.78" width="0.1524" layer="91"/>
@@
 <wire x1="-42.545" y1="45.4025" x2="-37.7825" y2="45.4025" width="0.1524" layer="91"/>
 </segment>
+<segment>
+<pinref part="IC1" gate="A1" pin="GND"/>
+<wire x1="-7.3025" y1="0.9525" x2="-7.3025" y2="-2.2225" width="0.1524" layer="91"/>
+</segment>
 </net>
 <net name="3VCC" class="0">
@@
 <segment>
 <pinref part="3.3REGULATOR" gate="G$1" pin="2"/>
-<pinref part="LM7805" gate="G$1" pin="IN"/>
 <wire x1="-27.94" y1="33.02" x2="-22.86" y2="33.02" width="0.1524" layer="91"/>
 <pinref part="BATTERY" gate="G$1" pin="2"/>
@@
 <wire x1="-42.545" y1="47.9425" x2="-27.94" y2="47.9425" width="0.1524" layer="91"/>
 <wire x1="-27.94" y1="47.9425" x2="-27.94" y2="33.02" width="0.1524" layer="91"/>
-</segment>
-</net>
+<pinref part="IC1" gate="A1" pin="VI"/>
+<wire x1="-17.4625" y1="8.5725" x2="-40.005" y2="8.5725" width="0.1524" layer="91"/>
+<wire x1="-40.005" y1="8.5725" x2="-40.005" y2="32.7025" width="0.1524" layer="91"/>
+<wire x1="-40.005" y1="32.7025" x2="-29.21" y2="32.7025" width="0.1524" layer="91"/>
+<wire x1="-29.21" y1="32.7025" x2="-29.21" y2="33.02" width="0.1524" layer="91"/>
+<wire x1="-29.21" y1="33.02" x2="-27.94" y2="33.02" width="0.1524" layer="91"/>
+</segment>
+</net>
